File: VocoreMotorShieldDRV8835.sch (EAGLE design)
At the start: 9 parts

Commit message: Version 0.2
Parts:
- removed JP7: (no value), pinhead:PINHD-1X8
- removed JP8: (no value), pinhead:PINHD-1X5
- JP4, JP5: device pinhead:PINHD-1X8 -> pinhead:PINHD-1X7
- JP6: device pinhead:PINHD-1X8 -> pinhead:PINHD-1X4
- renumbered U$1 to U1
Connections:
- removed net N$12: JP5.5, U1.G#24/LED2
- removed net N$15: JP5.8, U1.G#27/SPI_CS1
- removed net N$16: JP6.8, U1.G#14/PCM_TDX
- removed net N$17: JP6.7, U1.G#13/PCM_DRX
- removed net N$18: JP6.6, U1.G#12/PCM_CLK
- removed net N$19: JP6.5, U1.G#11/PCM_FS
- removed net N$20: JP6.4, U1.G#10/I2S_SDI/RXD
- removed net N$21: JP6.3, U1.G#09/I2S_SDO
- removed net N$22: JP6.1, JP6.2, U1.G#08/I2S_WS/TXD
- removed net N$23: JP7.1, U1.RESET
- removed net N$24: JP7.2, U1.G#00
- removed net N$25: JP7.3, U1.G#01/I2C_CLK
- removed net N$26: JP7.4, U1.G#02/I2C_SD
- removed net N$27: JP7.5, U1.G#03/SPI_CS0
- removed net N$28: JP7.6, U1.G#04/SPI_CLK
- removed net N$29: JP7.7, U1.G#05/SPI_MOSI
- removed net N$30: JP7.8, U1.G#06/SPI_MISO
- removed net N$31: JP8.2, U1.G#20/JTAG_TCLK
- removed net N$32: U1.G#19/JTAG_TMS
- removed net N$33: JP8.4, U1.G#18/JTAG_TDI
- removed net N$34: JP8.1, U1.G#21/JTAG_TRST
- removed net N$35: JP8.5, U1.G#17/JTAG_TDO
- net N$1: now also JP4.1, JP5.1; no longer JP4.5, JP4.6, JP4.7, JP4.8, U1.GND, U1.GND1, U1.GND3
- net N$10: now also JP5.4, JP6.1; no longer JP5.3, U1.G#22/LED0
- net N$11: now also JP5.3, JP6.2; no longer JP5.4, U1.G#23/LED1
- net N$13: now also JP5.5, JP6.4; no longer JP5.6, U1.G#25/LED3
- net N$14: now also JP5.6, JP6.3; no longer JP5.7, U1.G#26/LED4
- net N$2: now also JP5.2
- net N$3: now also JP4.2, JP4.7; no longer JP4.3, JP4.4, U1.+3.5V~+6.5V
- net N$4: now also JP4.3, U1.G#23/LED1; no longer JP4.1, U1.+1.8V
- net N$7: now also JP4.4, U1.G#24/LED2; no longer JP4.2, U1.+3.2V~+3.5VIN/OUT
- net N$8: now also JP4.5, U1.G#25/LED3; no longer JP5.1, U1.G#15/TXD2
- net N$9: now also JP4.6, U1.G#26/LED4; no longer JP5.2, U1.G#16/RXD2
Other:
- moved on the sheet: JP2, JP3
